File: PCB/Rev_1/LEOLED_rev1.kicad_pcb (KiCad board)
At the start: 2 copper layers, 70 x 40 mm, 91 parts, among them J1 PHEONIX_MPT_1725698, J2 USB_MicroB, J3 PHOENIX_MPT_1725656, J4 WURTH_61300411121, J5 FTSH-105-01-F-DV-K, J6 WURTH_61300211121, J7 PHOENIX_MPT_1725656, Q1 DMN65D8L-7, Q2 DMN65D8L-7, U1 BQ24210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

Commit message: layout edit
Parts:
- removed J6: WURTH_61300211121, Connector_Pin_Header:Pin_Header_Straight_1x02_Pitch2.54mm
- added R29: 0, Resistor_SMD:R_0805_2012Metric, F.Cu at (222.7, 108.7)
- R27, R28: moved to B.Cu
- moved D5 120.8 mm to (218.7, 132.3), turned to 270 degrees
- moved D3 119.2 mm to (218.7, 108.3), turned to 270 degrees
- moved D4 119.2 mm to (218.7, 120.3), turned to 270 degrees
- moved J7 111.1 mm to (221.0, 100.2), turned to 180 degrees
- moved R27 82.2 mm to (213.0, 113.3)
- moved R28 70.2 mm to (212.9, 102.1)
Routing:
- net Net-(D5-Pad2): track 0.00 -> 47.8 mm, vias 0 -> 2
- net Net-(D3-Pad1): track 0.00 -> 23.2 mm, vias 0 -> 2
- net Net-(D3-Pad2): track 0.00 -> 16.2 mm
- net Net-(D4-Pad2): track 0.00 -> 13.1 mm
- net /LED/LED_N: track 7.93 -> 14.1 mm
- net /LED/LED_P: track 0.00 -> 6.05 mm
- net GNDPWR: vias 0 -> 32
- added copper zone on B.Cu, net GNDPWR
- added copper zone on F.Cu, net GNDPWR
- added copper zone on F.Cu, net Net-(D3-Pad1)
- added copper zone on F.Cu, net Net-(D5-Pad2)
Other:
- board size 70 x 40 mm -> 84.1 x 40 mm
- net class Default: clearance 0.2 -> 0.254; trace_width 0.25 -> 0.254; via_dia 0.6 -> 1; via_drill 0.4 -> 0.5
- rule pad_to_mask_clearance: 0.2 -> 0
- rule trace_clearance: 0.2 -> 0.254
- rule trace_min: 0.2 -> 0.254
- rule via_min_drill: 0.3 -> 0.5
- rule via_min_size: 0.4 -> 1

Commit message: layout editing
Parts:
- moved TP15 29.1 mm to (198.0, 102.2)
- moved TP12 3.04 mm to (148.9, 110.0)
- moved TP11 2.64 mm to (150.9, 111.8)
- moved TP9 1.27 mm to (186.8, 108.3)
- moved TP8 0.51 mm to (149.1, 100.7)
Routing:
- net VDD: track 0.00 -> 99.5 mm, vias 0 -> 4
- net /Power/VUSB: track 0.00 -> 42.3 mm, vias 0 -> 2
- net /Power/NTC_P: track 0.00 -> 37.5 mm, vias 0 -> 1
- net /BLE/UART_TX: track 0.00 -> 37.2 mm, vias 0 -> 1
- net Net-(R21-Pad1): track 2.21 -> 37.5 mm, vias 0 -> 2
- net /BLE/UART_RX: track 0.00 -> 35.1 mm, vias 0 -> 2
- net /Power/BQ_CHG: track 0.00 -> 30.5 mm, vias 0 -> 2
- net Net-(R10-Pad1): track 0.00 -> 26.8 mm, vias 0 -> 2
- net /Power/SOLAR_VDD: track 0.00 -> 23.1 mm
- net /Power/BQ_PG: track 0.00 -> 22.5 mm, vias 0 -> 2
- net /Power/BQ_EN: track 0.00 -> 21.1 mm, vias 0 -> 2
- net /BLE/RESET: track 0.00 -> 19.5 mm, vias 0 -> 2
- net /Power/NTC_N: track 0.00 -> 17.3 mm, vias 0 -> 1
- net /BLE/SWO: track 0.00 -> 16.0 mm, vias 0 -> 2
- net GND: track 3.88 -> 19.6 mm, vias 0 -> 12
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Other:
- net class Default: clearance 0.254 -> 0.2; trace_width 0.254 -> 0.16
- rule trace_clearance: 0.254 -> 0.2
- rule trace_min: 0.254 -> 0.16
