File: PCB/Rev_1/LED.sch (KiCad schematic (older format))
At the start: 7 parts, among them J6 WURTH_61300211121, J7 PHOENIX_MPT_1725656

Commit message: layout edit
Parts:
- removed J6: WURTH_61300211121, Connector_Pin_Header:Pin_Header_Straight_1x02_Pitch2.54mm, symbol Connector_Pin_Header:WURTH_61300211121
- added R29: 0, Resistor_SMD:R_0805_2012Metric, symbol Resistor_SMD_0805:0
Connections:
- wire segments 29 -> 27
Changed lines of the file:
@@
 Wire Wire Line
 	4800 2200 4900 2200
-$Comp
-L Connector_Pin_Header:WURTH_61300211121 J6
-U 1 1 5B0437FB
-P 4000 2150
-F 0 "J6" H 4000 2250 50  0000 C CNN
-F 1 "WURTH_61300211121" H 4100 1900 50  0000 C CNN
-F 2 "Connector_Pin_Header:Pin_Header_Straight_1x02_Pitch2.54mm" H 4025 2350 60  0001 L CNN
-F 3 "http://katalog.we-online.de/em/datasheet/6130xx11121.pdf" H 4025 2450 60  0001 L CNN
-F 4 "3A, 250V" H 4025 2550 60  0001 L CNN "Rating"
-F 5 "NA" H 4025 2650 60  0001 L CNN "Tolerance"
-F 6 "Wurth Electronics Inc." H 4025 2750 60  0001 L CNN "Manufacturer"
-F 7 "61300211121" H 4025 2850 60  0001 L CNN "Manufacturer PN"
-F 8 "Digy-Key" H 4025 2950 60  0001 L CNN "Supplier"
-F 9 "732-5315-ND" H 4025 3050 60  0001 L CNN "Supplier PN"
-F 10 "https://www.digikey.com/products/en/connectors-interconnects/rectangular-connectors-headers-male-pins/314?k=&pkeyword=&pv88=2&FV=ffe0013a%2Cfffc02dc%2C1680001%2C8000010%2C1bf80001%2C1f700012%2C1f880152%2C1f9800e8%2C1fa40058&quantity=0&ColumnSort=0&page=1&pageSize=25" H 4025 3150 60  0001 L CNN "Supplier Link"
-F 11 "2 Positions Header Connector 0.100 (2.54mm) Through Hole Gold" H 4025 3250 60  0001 L CNN "Description"
-F 12 "Fitted" H 4025 3350 60  0001 L CNN "Assembly Option"
-	1    4000 2150
-	-1   0    0    1
-$EndComp
 Wire Wire Line
 	4650 1750 4650 1950
-Wire Wire Line
-	4200 2150 4400 2150
-Wire Wire Line
-	4400 2150 4400 2500
-Wire Wire Line
-	4400 2500 4650 2500
 Connection ~ 4650 2500
-Wire Wire Line
-	4200 2050 4400 2050
-Wire Wire Line
-	4400 2050 4400 1950
-Wire Wire Line
-	4400 1950 4650 1950
 Connection ~ 4650 1950
-$Comp
-L Connector_Terminal_Blocks:PHOENIX_MPT_1725656 J7
-U 1 1 5B044AC7
-P 6800 2400
-F 0 "J7" H 6800 2500 50  0000 C CNN
-F 1 "PHOENIX_MPT_1725656" H 6800 2200 50  0000 C CNN
-F 2 "Connector_Terminal_Blocks:TerminalBlock_Pheonix_MPT-2.54mm_2pol" H 6825 2600 60  0001 L CNN
-F 3 "https://media.digikey.com/pdf/Data%20Sheets/Phoenix%20Contact%20PDFs/1725656.pdf" H 6825 2700 60  0001 L CNN
-F 4 "6A, 125V" H 6825 2800 60  0001 L CNN "Rating"
-F 5 "NA" H 6825 2900 60  0001 L CNN "Tolerance"
-F 6 "Phoenix Contact" H 6825 3000 60  0001 L CNN "Manufacturer"
-F 7 "1725656" H 6825 3100 60  0001 L CNN "Manufacturer PN"
-F 8 "Digy-Key" H 6825 3200 60  0001 L CNN "Supplier"
-F 9 "277-1273-ND" H 6825 3300 60  0001 L CNN "Supplier PN"
-F 10 "https://www.digikey.com/product-detail/en/phoenix-contact/1725656/277-1273-ND/267462" H 6825 3400 60  0001 L CNN "Supplier Link"
-F 11 "2 Position Wire to Board Terminal Block Horizontal with Board 0.100 (2.54mm) Through Hole" H 6825 3500 60  0001 L CNN "Description"
-F 12 "Fitted" H 6825 3600 60  0001 L CNN "Assembly Option"
-	1    6800 2400
-	1    0    0    -1
-$EndComp
 Wire Wire Line
 	6600 2400 6250 2400
@@
 Text HLabel 7150 3600 2    50   Input ~ 0
 LED_N
+$Comp
+L Connector_Terminal_Blocks:PHOENIX_MPT_1725656 J7
+U 1 1 5B044AC7
+P 6800 2400
+F 0 "J7" H 6800 2500 50  0000 C CNN
+F 1 "PHOENIX_MPT_1725656" H 6800 2200 50  0000 C CNN
+F 2 "Connector_Terminal_Blocks:TerminalBlock_Pheonix_MPT-2.54mm_2pol" H 6825 2600 60  0001 L CNN
+F 3 "https://media.digikey.com/pdf/Data%20Sheets/Phoenix%20Contact%20PDFs/1725656.pdf" H 6825 2700 60  0001 L CNN
+F 4 "6A, 125V" H 6825 2800 60  0001 L CNN "Rating"
+F 5 "NA" H 6825 2900 60  0001 L CNN "Tolerance"
+F 6 "Phoenix Contact" H 6825 3000 60  0001 L CNN "Manufacturer"
+F 7 "1725656" H 6825 3100 60  0001 L CNN "Manufacturer PN"
+F 8 "Digy-Key" H 6825 3200 60  0001 L CNN "Supplier"
+F 9 "277-1273-ND" H 6825 3300 60  0001 L CNN "Supplier PN"
+F 10 "https://www.digikey.com/product-detail/en/phoenix-contact/1725656/277-1273-ND/267462" H 6825 3400 60  0001 L CNN "Supplier Link"
+F 11 "2 Position Wire to Board Terminal Block Horizontal with Board 0.100 (2.54mm) Through Hole" H 6825 3500 60  0001 L CNN "Description"
+F 12 "Fitted" H 6825 3600 60  0001 L CNN "Assembly Option"
+	1    6800 2400
+	1    0    0    -1
+$EndComp
+$Comp
+L Resistor_SMD_0805:0 R29
+U 1 1 5B341C22
+P 4100 2200
+F 0 "R29" V 3893 2200 50  0000 C CNN
+F 1 "0" V 3984 2200 50  0000 C CNN
+F 2 "Resistor_SMD:R_0805_2012Metric" H 4125 2400 60  0001 L CNN
+F 3 "http://industrial.panasonic.com/www-cgi/jvcr13pz.cgi?E+PZ+3+AOA0001+ERJ6GEY0R00V+7+WW" H 4125 2500 60  0001 L CNN
+F 4 "0.125W" H 4125 2600 60  0001 L CNN "Rating"
+F 5 "NA" H 4125 2700 60  0001 L CNN "Tolerance"
+F 6 "Panasonic Electronic Component" H 4125 2800 60  0001 L CNN "Manufacturer"
+F 7 "ERJ-6GEY0R00V" H 4125 2900 60  0001 L CNN "Manufacturer PN"
+F 8 "Digy-Key" H 4125 3000 60  0001 L CNN "Supplier"
+F 9 "P0.0ACT-ND" H 4125 3100 60  0001 L CNN "Supplier PN"
+F 10 "https://www.digikey.com/product-detail/en/panasonic-electronic-components/ERJ-6GEY0R00V/P0.0ACT-ND/82955" H 4125 3200 60  0001 L CNN "Supplier Link"
+F 11 "0 Ohms Jumper 0.125W, 1/8W Chip Resistor 0805 (2012 Metric) Automotive AEC-Q200 Thick Film" H 4125 3300 60  0001 L CNN "Description"
+F 12 "Not Fitted" H 4200 2250 60  0000 L CNN "Assembly Option"
+	1    4100 2200
+	-1   0    0    1
+$EndComp
+Wire Wire Line
+	4100 2500 4100 2350
+Wire Wire Line
+	4100 2500 4650 2500
+Wire Wire Line
+	4100 2050 4100 1950
+Wire Wire Line
+	4100 1950 4650 1950
 $EndSCHEMATC

Commit message: cleaning up
Parts:
- R27, R28: Assembly Option Fitted -> Not Fitted
Changed lines of the file:
@@
 F 10 "https://www.digikey.com/product-detail/en/panasonic-electronic-components/ERJ-6GEY0R00V/P0.0ACT-ND/82955" H 6625 2750 60  0001 L CNN "Supplier Link"
 F 11 "0 Ohms Jumper 0.125W, 1/8W Chip Resistor 0805 (2012 Metric) Automotive AEC-Q200 Thick Film" H 6625 2850 60  0001 L CNN "Description"
-F 12 "Fitted" H 6625 2950 60  0001 L CNN "Assembly Option"
+F 12 "Not Fitted" V 6750 1650 60  0000 L CNN "Assembly Option"
 	1    6600 1750
 	0    1    1    0
@@
 F 10 "https://www.digikey.com/product-detail/en/panasonic-electronic-components/ERJ-6GEY0R00V/P0.0ACT-ND/82955" H 6675 4600 60  0001 L CNN "Supplier Link"
 F 11 "0 Ohms Jumper 0.125W, 1/8W Chip Resistor 0805 (2012 Metric) Automotive AEC-Q200 Thick Film" H 6675 4700 60  0001 L CNN "Description"
-F 12 "Fitted" H 6675 4800 60  0001 L CNN "Assembly Option"
+F 12 "Not Fitted" V 6800 3550 60  0000 L CNN "Assembly Option"
 	1    6650 3600
 	0    1    1    0
