File: PCB/Rev_1/Power.sch (KiCad schematic (older format))
At the start: 47 parts, among them Q1 DMN65D8L-7, Q2 DMN65D8L-7, U1 BQ24210, U2 MAX1725

Commit message: layout editing
Changed lines of the file:
@@
 $EndComp
-Wire Wire Line
-	9850 1400 9850 1450
 Wire Wire Line
 	8750 1950 9850 1950
@@
 Wire Wire Line
 	9500 1100 9850 1100
-Connection ~ 9850 1450
-Wire Wire Line
-	9850 1450 9850 1950
 Connection ~ 9850 1100
 Wire Wire Line
 	9850 1100 10050 1100
+Wire Wire Line
+	9850 1400 9850 1950
 $EndSCHEMATC

Commit message: cleaning up
Parts:
- TH1: Assembly Option Fitted -> Not Fitted
Changed lines of the file:
@@
 F 10 "https://www.digikey.com/product-detail/en/tdk-corporation/NTCG164KF104FT1/445-2556-1-ND/934255" H 8925 5700 60  0001 L CNN "Supplier Link"
 F 11 "NTC Thermistor 100k 0603 (1608 Metric)" H 8925 5800 60  0001 L CNN "Description"
-F 12 "Fitted" H 8925 5900 60  0001 L CNN "Assembly Option"
+F 12 "Not Fitted" H 8400 4900 60  0000 L CNN "Assembly Option"
 	1    8900 4700
 	1    0    0    -1
